File: MeterMaker/Metermaker.kicad_pcb (KiCad board)
At the start: 2 copper layers, 100 x 100 mm, 135 parts, among them J1 Barrel_Jack_Switch, J10 Bornier, J11 Bornier, J12 Bornier, J13 Bornier, J14 Bornier, J15 Hole, J16 Hole, J2 Bornier, J3 Bornier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

Commit message: Added initial code
Parts:
- added R60: 10k, Resistor_THT:R_Axial_DIN0207_L6.3mm_D2.5mm_P7.62mm_Horizontal, F.Cu at (145.8, 93.5)
- added R61: 10k, Resistor_THT:R_Axial_DIN0207_L6.3mm_D2.5mm_P7.62mm_Horizontal, F.Cu at (133.3, 85.6)
- added R62: 10k, Resistor_THT:R_Axial_DIN0207_L6.3mm_D2.5mm_P7.62mm_Horizontal, F.Cu at (119.1, 85.6)
- added R63: 10k, Resistor_THT:R_Axial_DIN0207_L6.3mm_D2.5mm_P7.62mm_Horizontal, F.Cu at (101.9, 84.6)
- added R64: 10k, Resistor_THT:R_Axial_DIN0207_L6.3mm_D2.5mm_P7.62mm_Horizontal, F.Cu at (101.9, 81.3)
- C10, C7, C8: value 100 nF, 100 V -> 100 nF
- R22, R23, R24, R25, R26: value 10k -> 1k
- moved C20 12.8 mm to (86.6, 75.9)
- moved R35 9.78 mm to (96.5, 80.2)
- moved R37 9.71 mm to (96.5, 83.6)
- moved R10 8.54 mm to (110.9, 139.0), turned to 0 degrees
- moved R11 8.46 mm to (110.9, 135.6), turned to 0 degrees
- moved C8 7.59 mm to (117.6, 132.3), turned to 180 degrees
- moved C18 6.51 mm to (86.1, 79.8)
- moved R23 5.41 mm to (115.6, 85.3)
- moved R13 5.05 mm to (137.2, 138.8), turned to 0 degrees
- moved R14 4.47 mm to (145.0, 135.4), turned to 180 degrees
- moved R9 4.22 mm to (95.5, 139.2), turned to 90 degrees
- moved C7 3.84 mm to (88.4, 135.7), turned to 90 degrees
- moved R8 3.48 mm to (92.2, 131.6), turned to -90 degrees
- moved RV1 1.61 mm to (147.2, 66.1)
- moved R25 1.42 mm to (129.8, 85.8)
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Connections:
- C10 pad 1: Net-(J5-Pin_2) -> Net-(C10-Pad1)
- C10 pad 2: Net-(C10-Pad2) -> Net-(J5-Pin_1)
- C7 pad 1: Net-(J2-Pin_2) -> Net-(C7-Pad1)
- C7 pad 2: Net-(C7-Pad2) -> Net-(J2-Pin_1)
- C8 pad 1: Net-(J4-Pin_1) -> Net-(C8-Pad1)
- C8 pad 2: Net-(C8-Pad2) -> Net-(J3-Pin_2)
- R10 pad 1: Net-(C8-Pad2) -> Net-(J4-Pin_1)
- R10 pad 2: Net-(J3-Pin_2) -> Net-(C8-Pad1)
- R11 pad 2: Net-(J3-Pin_2) -> Net-(C8-Pad1)
- R13 pad 1: Net-(C10-Pad2) -> Net-(J5-Pin_2)
- R13 pad 2: Net-(J5-Pin_1) -> Net-(C10-Pad1)
- R14 pad 2: Net-(J5-Pin_1) -> Net-(C10-Pad1)
- R8 pad 2: Net-(J2-Pin_1) -> Net-(C7-Pad1)
- R9 pad 1: Net-(C7-Pad2) -> Net-(J2-Pin_2)
- R9 pad 2: Net-(J2-Pin_1) -> Net-(C7-Pad1)
- SW1 pad 2: Net-(R23-Pad2) -> Net-(R64-Pad1)
- SW2 pad 2: Net-(R22-Pad2) -> Net-(R60-Pad1)
- SW3 pad 2: Net-(R24-Pad2) -> Net-(R63-Pad1)
- SW4 pad 2: Net-(R25-Pad2) -> Net-(R62-Pad1)
- SW5 pad 2: Net-(R26-Pad2) -> Net-(R61-Pad1)
Routing:
- net Net-(R23-Pad2): track 36.2 -> 14.0 mm
- net Net-(R26-Pad2): track 45.2 -> 24.6 mm
- net Net-(R64-Pad1): track 0.00 -> 15.5 mm
- net Net-(C7-Pad1): track 0.00 -> 14.3 mm
- net Net-(C10-Pad1): track 0.00 -> 14.3 mm
- net Net-(R63-Pad1): track 0.00 -> 12.5 mm
- net Net-(R60-Pad1): track 0.00 -> 11.9 mm
- net Net-(R22-Pad2): track 52.7 -> 40.9 mm
- net Net-(R62-Pad1): track 0.00 -> 11.3 mm
- net Net-(R61-Pad1): track 0.00 -> 11.2 mm
- net DAC3: track 46.6 -> 35.4 mm
- net Net-(J5-Pin_1): track 28.0 -> 17.3 mm
- net Net-(R24-Pad2): track 32.6 -> 22.3 mm
- net Net-(C8-Pad1): track 0.00 -> 7.12 mm
- net Net-(R25-Pad2): track 27.0 -> 20.1 mm
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Other:
- board text added: "METERMAKER BY DANIEL MARKS CC-BY-SA 4.0 VERSION 2"
- board text removed: "METERMAKER BY DANIEL MARKS CC-BY-SA 4.0 VERSION 1"
