File: MeterMaker/Metermaker.kicad_sch (KiCad schematic)
At the start: 135 parts, among them J1 Barrel_Jack_Switch, J10 Bornier, J11 Bornier, J12 Bornier, J13 Bornier, J14 Bornier, J15 Hole, J16 Hole, J2 Bornier, J3 Bornier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

Commit message: Added initial code
Parts:
- added R60, R61, R62, R63, R64: 10k, Resistor_THT:R_Axial_DIN0207_L6.3mm_D2.5mm_P7.62mm_Horizontal, symbol Device:R
- C10, C7, C8: value 100 nF, 100 V -> 100 nF
- R22, R23, R24, R25, R26: value 10k -> 1k
Connections:
- net at R13.1: now also J5.2 (Pin_2); no longer C10.2
- net at R13.2, R14.2: now also C10.1; no longer J5.1 (Pin_1), R15.1
- net at C7.1: now also R8.2, R9.2; no longer J2.2 (Pin_2)
- net at C7.2: now also J2.1 (Pin_1), R7.1; no longer R9.1
- net at R26.2, U4.9: now also R61.2; no longer SW5.2
- net at J3.2 (Pin_2), R12.1: now also C8.2; no longer R10.2, R11.2
- net at J4.1 (Pin_1): now also R10.1; no longer C8.1
- net at R25.2, U4.5: now also R62.2; no longer SW4.2
- net at R24.2, U4.3: now also R63.2; no longer SW3.2
- net at R23.2, U4.1: now also R64.2; no longer SW1.2
- net at R22.2, U4.11: now also R60.2; no longer SW2.2
- new net: R61.1, SW5.2
- new net: C8.1, R10.2, R11.2
- new net: R60.1, SW2.2
- new net: R62.1, SW4.2
- new net: C10.2, J5.1 (Pin_1), R15.1
- new net: J2.2 (Pin_2), R9.1
- new net: R63.1, SW3.2
- new net: R64.1, SW1.2
Other:
- moved on the sheet: C10, C7, C8, R10, R11, R13, R14, R23, R25, R26, R8, R9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
